Commit message: Fix typo in mimic joint name (gripper).

File: gomtec_robot_description/urdf/Gripper_macro.xacro (robot description, xacro)
@@ -88,5 +88,5 @@
             <axis xyz="0 1 0" />
             <limit effort="0" lower="0" upper="0.035" velocity="0.05" />
-            <mimic joint="${prefix}joint_gl_linear" />
+            <mimic joint="${prefix}joint_f1_linear" />
         </joint>
         <joint name="${prefix}joint_tcp" type="fixed">

File: gomtec_robot_description/urdf/Roberta_P80_800.urdf (robot description, URDF)
Before this commit: robot Roberta_P80_800, 12 links, 11 joints
Joints:
- joint joint_f2_linear: mimic joint=joint_gl_linear -> joint=joint_f1_linear
