Commit message: Fixed gripper orientation: gripper and camera gripper mounting orientation to the arm was twisted by 90°

File: gomtec_robot_description/urdf/CameraGripper_macro.xacro (robot description, xacro)
@@ -6,5 +6,5 @@
         <link name="${prefix}link_Gripper">
             <visual>
-                <origin xyz="0 0 0.0315" rpy="${pi/2} 0 ${pi/2}" />
+                <origin xyz="0 0 0.0315" rpy="${pi/2} 0 0" />
                 <geometry>
                     <mesh
@@ -17,5 +17,5 @@
             </visual>
             <collision>
-                <origin xyz="0 0 0.0315" rpy="${pi/2} 0 ${pi/2}" />
+                <origin xyz="0 0 0.0315" rpy="${pi/2} 0 0" />
                 <geometry>
                     <mesh
@@ -27,5 +27,5 @@
         <link name="${prefix}link_Finger1">
             <visual>
-                <origin xyz="0 -0.00323 0" rpy="${pi/2} 0 ${-pi/2}" />
+                <origin xyz="-0.00323 0 0" rpy="${pi/2} 0 ${-pi}" />
                 <geometry>
                     <mesh
@@ -38,5 +38,5 @@
             </visual>
             <collision>
-                <origin xyz="0 -0.00323 0" rpy="${pi/2} 0 ${-pi/2}" />
+                <origin xyz="-0.00323 0 0" rpy="${pi/2} 0 ${-pi}" />
                 <geometry>
                     <mesh
@@ -48,5 +48,5 @@
         <link name="${prefix}link_Finger2">
             <visual>
-                <origin xyz="0 0.00323 0" rpy="${pi/2} 0 ${pi/2}" />
+                <origin xyz="0.00323 0 0" rpy="${pi/2} 0 0" />
                 <geometry>
                     <mesh
@@ -59,5 +59,5 @@
             </visual>
             <collision>
-                <origin xyz="0 0.00323 0" rpy="${pi/2} 0 ${pi/2}" />
+                <origin xyz="0.00323 0 0" rpy="${pi/2} 0 0" />
                 <geometry>
                     <mesh
@@ -79,5 +79,5 @@
             <child link="${prefix}link_Finger1" />
             <origin xyz="0 0 0.141" rpy="0 0 0" />
-            <axis xyz="0 -1 0" />
+            <axis xyz="-1 0 0" />
             <limit effort="0" lower="0" upper="0.035" velocity="0.05" />
         </joint>
@@ -86,7 +86,7 @@
             <child link="${prefix}link_Finger2" />
             <origin xyz="0 0 0.141" rpy="0 0 0" />
-            <axis xyz="0 1 0" />
+            <axis xyz="1 0 0" />
             <limit effort="0" lower="0" upper="0.035" velocity="0.05" />
-            <mimic joint="${prefix}joint_gl_linear" />
+            <mimic joint="${prefix}joint_f1_linear" />
         </joint>
         <joint name="${prefix}joint_tcp" type="fixed">

File: gomtec_robot_description/urdf/Gripper_macro.xacro (robot description, xacro)
@@ -6,5 +6,5 @@
         <link name="${prefix}link_Gripper">
             <visual>
-                <origin xyz="0 0 0.0315" rpy="${pi/2} 0 ${pi/2}" />
+                <origin xyz="0 0 0.0315" rpy="${pi/2} 0 0" />
                 <geometry>
                     <mesh
@@ -17,5 +17,5 @@
             </visual>
             <collision>
-                <origin xyz="0 0 0.0315" rpy="${pi/2} 0 ${pi/2}" />
+                <origin xyz="0 0 0.0315" rpy="${pi/2} 0 0" />
                 <geometry>
                     <mesh
@@ -27,5 +27,5 @@
         <link name="${prefix}link_Finger1">
             <visual>
-                <origin xyz="0 -0.00323 0" rpy="${pi/2} 0 ${-pi/2}" />
+                <origin xyz="-0.00323 0 0" rpy="${pi/2} 0 ${-pi}" />
                 <geometry>
                     <mesh
@@ -38,5 +38,5 @@
             </visual>
             <collision>
-                <origin xyz="0 -0.00323 0" rpy="${pi/2} 0 ${-pi/2}" />
+                <origin xyz="-0.00323 0 0" rpy="${pi/2} 0 ${-pi}" />
                 <geometry>
                     <mesh
@@ -48,5 +48,5 @@
         <link name="${prefix}link_Finger2">
             <visual>
-                <origin xyz="0 0.00323 0" rpy="${pi/2} 0 ${pi/2}" />
+                <origin xyz="0.00323 0 0" rpy="${pi/2} 0 0" />
                 <geometry>
                     <mesh
@@ -59,5 +59,5 @@
             </visual>
             <collision>
-                <origin xyz="0 0.00323 0" rpy="${pi/2} 0 ${pi/2}" />
+                <origin xyz="0.00323 0 0" rpy="${pi/2} 0 0" />
                 <geometry>
                     <mesh
@@ -79,5 +79,5 @@
             <child link="${prefix}link_Finger1" />
             <origin xyz="0 0 0.141" rpy="0 0 0" />
-            <axis xyz="0 -1 0" />
+            <axis xyz="-1 0 0" />
             <limit effort="0" lower="0" upper="0.035" velocity="0.05" />
         </joint>
@@ -86,5 +86,5 @@
             <child link="${prefix}link_Finger2" />
             <origin xyz="0 0 0.141" rpy="0 0 0" />
-            <axis xyz="0 1 0" />
+            <axis xyz="1 0 0" />
             <limit effort="0" lower="0" upper="0.035" velocity="0.05" />
             <mimic joint="${prefix}joint_f1_linear" />

File: gomtec_robot_description/urdf/Roberta_P80_800.urdf (robot description, URDF)
Before this commit: robot Roberta_P80_800, 12 links, 11 joints
Joints:
- joint joint_f1_linear: axis 0 -1 0 -> -1 0 0
- joint joint_f2_linear: axis 0 1 0 -> 1 0 0
