Commit message: masterthesis Abbas Khoobyari

File: gomtec_robot_description/urdf/P80_800_macro.xacro (robot description, xacro)
@@ -6,5 +6,5 @@
         <link name="${prefix}base_link">
             <visual>
-                <origin xyz="0 0 0" rpy="${pi/2} 0 0" />
+                <origin xyz="0 0 0.11" rpy="${pi} 0 0" />
                 <geometry>
                     <mesh
@@ -12,10 +12,10 @@
                         scale="0.001 0.001 0.001" />
                 </geometry>
-                <material name="gomtec_silver">
-                    <color rgba="0.5 0.5 0.5 1" />
-                </material>
-            </visual>
-            <collision>
-                <origin xyz="0 0 0" rpy="${pi/2} 0 0" />
+                <material name="gomtec_dunkel">
+                    <color rgba="0.4 0.4 0.4 1" />
+                </material>
+            </visual>
+            <collision>
+                <origin xyz="0 0 0.11" rpy="${pi} 0 0" />
                 <geometry>
                     <mesh
@@ -27,5 +27,5 @@
         <link name="${prefix}link_1">
             <visual>
-                <origin xyz="0 0 -0.082" rpy="${pi/2} 0 ${-pi/2}" />
+                <origin xyz="0 0 0" rpy="${pi} 0 ${pi}" />
                 <geometry>
                     <mesh
@@ -33,10 +33,10 @@
                         scale="0.001 0.001 0.001" />
                 </geometry>
-                <material name="gomtec_black">
-                    <color rgba="0.15 0.15 0.15 1" />
-                </material>
-            </visual>
-            <collision>
-                <origin xyz="0 0 -0.082" rpy="${pi/2} 0 ${-pi/2}" />
+                <material name="gomtec_grau">
+                    <color rgba="0.6 0.6 0.5 1" />
+                </material>
+            </visual>
+            <collision>
+                <origin xyz="0 0 0" rpy="${pi} 0 ${pi}" />
                 <geometry>
                     <mesh
@@ -48,5 +48,5 @@
         <link name="${prefix}link_2">
             <visual>
-                <origin xyz="0 0.08025 0" rpy="${pi/2} 0 ${pi/2}" />
+                <origin xyz="0 0.135 0.01" rpy="${-pi} ${-pi/2} ${pi/2}" />
                 <geometry>
                     <mesh
@@ -54,10 +54,10 @@
                         scale="0.001 0.001 0.001" />
                 </geometry>
-                <material name="gomtec_black">
-                    <color rgba="0.15 0.15 0.15 1" />
-                </material>
-            </visual>
-            <collision>
-                <origin xyz="0 0.08025 0" rpy="${pi/2} 0 ${pi/2}" />
+                <material name="gomtec_grau">
+                    <color rgba="0.6 0.6 0.5 1" />
+                </material>
+            </visual>
+            <collision>
+                <origin xyz="0 0.135 0.01" rpy="${-pi} ${-pi/2} ${pi/2}" />
                 <geometry>
                     <mesh
@@ -69,5 +69,5 @@
         <link name="${prefix}link_3">
             <visual>
-                <origin xyz="0 0 0.075" rpy="${-pi/2} 0 ${-pi/2}" />
+                <origin xyz="0 0.1 -0.02" rpy="${-pi/2} 0 0" />
                 <geometry>
                     <mesh
@@ -75,10 +75,10 @@
                         scale="0.001 0.001 0.001" />
                 </geometry>
-                <material name="gomtec_black">
-                    <color rgba="0.15 0.15 0.15 1" />
-                </material>
-            </visual>
-            <collision>
-                <origin xyz="0 0 0.075" rpy="${-pi/2} 0 ${-pi/2}" />
+                <material name="gomtec_grau">
+                    <color rgba="0.6 0.6 0.5 1" />
+                </material>
+            </visual>
+            <collision>
+                <origin xyz="0 0.1 -0.02" rpy="${-pi/2} 0 0" />
                 <geometry>
                     <mesh
@@ -90,5 +90,5 @@
         <link name="${prefix}link_4">
             <visual>
-                <origin xyz="0 0.0655 0.28" rpy="${-pi/2} 0 ${pi/2}" />
+                <origin xyz="0.25 -0.0115 -0.005" rpy="0 ${-pi/2} 0" />
                 <geometry>
                     <mesh
@@ -96,10 +96,10 @@
                         scale="0.001 0.001 0.001" />
                 </geometry>
-                <material name="gomtec_black">
-                    <color rgba="0.15 0.15 0.15 1" />
-                </material>
-            </visual>
-            <collision>
-                <origin xyz="0 0.0655 0.28" rpy="${-pi/2} 0 ${pi/2}" />
+                <material name="gomtec_grau">
+                    <color rgba="0.6 0.6 0.5 1" />
+                </material>
+            </visual>
+            <collision>
+                <origin xyz="0.25 -0.0115 -0.005" rpy="0 ${-pi/2} 0" />
                 <geometry>
                     <mesh
@@ -111,5 +111,5 @@
         <link name="${prefix}link_5">
             <visual>
-                <origin xyz="0 0 0.0665" rpy="${-pi/2} 0 ${-pi/2}" />
+                <origin xyz="0 0 0.007" rpy="${-pi/2} 0 ${-pi}" />
                 <geometry>
                     <mesh
@@ -117,10 +117,10 @@
                         scale="0.001 0.001 0.001" />
                 </geometry>
-                <material name="gomtec_black">
-                    <color rgba="0.15 0.15 0.15 1" />
-                </material>
-            </visual>
-            <collision>
-                <origin xyz="0 0 0.0665" rpy="${-pi/2} 0 ${-pi/2}" />
+               <material name="gomtec_grau">
+                    <color rgba="0.6 0.6 0.5 1" />
+                </material>
+            </visual>
+            <collision>
+                <origin xyz="0 0 0.007" rpy="${-pi/2} 0 ${-pi}" />
                 <geometry>
                     <mesh
@@ -143,5 +143,5 @@
             <parent link="${prefix}link_1" />
             <child link="${prefix}link_2" />
-            <origin rpy="0 0 0" xyz="0 0 0" />
+            <origin rpy="0 0 0" xyz="0 0 0.45" />
             <axis xyz="0 1 0" />
             <limit effort="0" velocity="${100*pi/180}"/>
@@ -157,6 +157,6 @@
             <parent link="${prefix}link_3" />
             <child link="${prefix}link_4" />
-            <origin rpy="0 0 0" xyz="0 0 0" />
-            <axis xyz="0 0 1" />
+            <origin rpy="0 0 0" xyz="0 0.025 -0.01" />
+            <axis xyz="1 0 0" />
             <limit effort="0" velocity="${100*pi/180}"/>
         </joint>
@@ -164,6 +164,6 @@
             <parent link="${prefix}link_4" />
             <child link="${prefix}link_5" />
-            <origin rpy="0 0 0" xyz="0 0 0.42" />
-            <axis xyz="0 -1 0" />
+            <origin rpy="0 0 0" xyz="0.30 0.005 -0.006" />
+            <axis xyz="0 1 0" />
             <limit effort="0" velocity="${200*pi/180}"/>
         </joint>
@@ -171,6 +171,6 @@
             <parent link="${prefix}link_5" />
             <child link="${prefix}link_flange" />
-            <origin rpy="0 0 0" xyz="0 0 0.112" />
-            <axis xyz="0 0 1" />
+            <origin rpy="0 0 0" xyz="0.07 -0.002 0.000" />
+            <axis xyz="1 0 0" />
             <limit effort="0" velocity="${200*pi/180}" />
         </joint>

File: gomtec_robot_description/urdf/Roberta_P80_800.urdf (robot description, URDF)
Before this commit: robot Roberta_P80_800, 12 links, 11 joints
Links:
- added link cameralink; collision mesh filename=package://gomtec_robot_description/meshes/collision/kinect_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; visual mesh filename=package://gomtec_robot_description/meshes/visual/kinect_cam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
- added link depth_frame
- added link depth_optical_frame
- added link rgb_frame
- added link rgb_optical_frame
Joints:
- added joint depth_joint: type fixed, parent cameralink, child depth_frame, origin xyz=0.0 -0.02 0.0 rpy=0 0 0
- added joint depth_optical_joint: type fixed, parent depth_frame, child depth_optical_frame, origin xyz=0 0 0 rpy=-1.57079632679 0.0 -1.57079632679
- added joint joint: type fixed, parent link_RoboCommander, child cameralink
- added joint rgb_joint: type fixed, parent cameralink, child rgb_frame, origin xyz=0.0 -0.0125 0.0 rpy=0 0 0
- added joint rgb_optical_joint: type fixed, parent rgb_frame, child rgb_optical_frame, origin xyz=0 0 0 rpy=-1.57079632679 0.0 -1.57079632679
- joint joint_2: origin xyz=0 0 0 rpy=0 0 0 -> xyz=0 0 0.45 rpy=0 0 0
- joint joint_4: axis 0 0 1 -> 1 0 0; origin xyz=0 0 0 rpy=0 0 0 -> xyz=0 0.025 -0.01 rpy=0 0 0
- joint joint_5: axis 0 -1 0 -> 0 1 0; origin xyz=0 0 0.42 rpy=0 0 0 -> xyz=0.30 0.005 -0.006 rpy=0 0 0
- joint joint_6: axis 0 0 1 -> 1 0 0; origin xyz=0 0 0.112 rpy=0 0 0 -> xyz=0.07 -0.002 0.000 rpy=0 0 0
- joint joint_GripperBase: origin xyz=0 0 0 rpy=0 0 0 -> xyz=0.1 0 -0.1 rpy=0 0 0
- joint joint_f1_linear: axis -1 0 0 -> 0 0 1; origin xyz=0 0 0.141 rpy=0 0 0 -> xyz=0.1 0 0 rpy=0 0 0
- joint joint_f2_linear: axis 1 0 0 -> 0 0 -1; origin xyz=0 0 0.141 rpy=0 0 0 -> xyz=0.1 0 0.07 rpy=0 0 0
- joint joint_tcp: origin xyz=0 0 0.141 rpy=0 0 0 -> xyz=0 0 0 rpy=0 0 0

File: gomtec_robot_description/urdf/Roberta_P80_800.xacro (robot description, xacro)
@@ -7,4 +7,6 @@
 	<xacro:include filename="$(find gomtec_robot_description)/urdf/Gripper_macro.xacro"/>
 	<xacro:Gripper prefix="" flange_link="link_RoboCommander"/>
+        <xacro:include filename="$(find gomtec_robot_description)/urdf/kinect_camera.urdf.xacro"/>
+	<xacro:kinect_camera_model prefix="" flange_link="link_RoboCommander"/>
 	<!--include filename="$(find gomtec_robot_description)/urdf/CameraGripper_macro.xacro"/>
 	<xacro:CameraGripper prefix="" flange_link="link_RoboCommander"/-->

File: gomtec_robot_description/urdf/Roberta_P80_800_Vision.urdf (robot description, URDF)
Before this commit: robot Roberta_P80_800, 12 links, 11 joints
Links:
- added link cameralink; collision mesh filename=package://gomtec_robot_description/meshes/collision/kinect_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; visual mesh filename=package://gomtec_robot_description/meshes/visual/kinect_cam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
- added link depth_frame
- added link depth_optical_frame
- added link rgb_frame
- added link rgb_optical_frame
Joints:
- added joint depth_joint: type fixed, parent cameralink, child depth_frame, origin xyz=0.0 -0.02 0.0 rpy=0 0 0
- added joint depth_optical_joint: type fixed, parent depth_frame, child depth_optical_frame, origin xyz=0 0 0 rpy=-1.57079632679 0.0 -1.57079632679
- added joint joint: type fixed, parent link_RoboCommander, child cameralink
- added joint rgb_joint: type fixed, parent cameralink, child rgb_frame, origin xyz=0.0 -0.0125 0.0 rpy=0 0 0
- added joint rgb_optical_joint: type fixed, parent rgb_frame, child rgb_optical_frame, origin xyz=0 0 0 rpy=-1.57079632679 0.0 -1.57079632679
- joint joint_2: origin xyz=0 0 0 rpy=0 0 0 -> xyz=0 0 0.45 rpy=0 0 0
- joint joint_4: axis 0 0 1 -> 1 0 0; origin xyz=0 0 0 rpy=0 0 0 -> xyz=0 0.025 -0.01 rpy=0 0 0
- joint joint_5: axis 0 -1 0 -> 0 1 0; origin xyz=0 0 0.42 rpy=0 0 0 -> xyz=0.30 0.005 -0.006 rpy=0 0 0
- joint joint_6: axis 0 0 1 -> 1 0 0; origin xyz=0 0 0.112 rpy=0 0 0 -> xyz=0.07 -0.002 0.000 rpy=0 0 0
- joint joint_GripperBase: origin xyz=0 0 0 rpy=0 0 0 -> xyz=0.1 0 -0.1 rpy=0 0 0
- joint joint_f1_linear: axis -1 0 0 -> 0 0 1; origin xyz=0 0 0.141 rpy=0 0 0 -> xyz=0.1 0 0 rpy=0 0 0
- joint joint_f2_linear: axis 1 0 0 -> 0 0 -1; origin xyz=0 0 0.141 rpy=0 0 0 -> xyz=0.1 0 0.07 rpy=0 0 0
- joint joint_tcp: origin xyz=0 0 0.141 rpy=0 0 0 -> xyz=0 0 -0.141 rpy=0 0 0

File: gomtec_robot_description/urdf/Roberta_P80_800_Vision.xacro (robot description, xacro)
@@ -7,3 +7,5 @@
 	<include filename="$(find gomtec_robot_description)/urdf/CameraGripper_macro.xacro"/>
 	<xacro:CameraGripper prefix="" flange_link="link_RoboCommander"/>
+	<xacro:include filename="$(find gomtec_robot_description)/urdf/kinect_camera.urdf.xacro"/>
+	<xacro:kinect_camera_model prefix="" flange_link="link_RoboCommander"/>
 </robot>
